File: 8xrj45.kicad_pcb (KiCad board)
At the start: 2 copper layers, 5 parts, among them j1 Conn_01x40

Commit message: v2 design
Routing:
- net GND: track 133.3 -> 0.00 mm
- net Net-(c3_4-Pad5): track 76.3 -> 158.0 mm, vias 2 -> 0
- net Net-(c3_4-Pad3): track 61.6 -> 79.8 mm
- net Net-(c5_6-Pad13): track 57.5 -> 70.7 mm
- net Net-(c7_8-Pad16): track 116.2 -> 126.2 mm
- net Net-(c7_8-Pad14): track 117.9 -> 126.0 mm
- net +5V: track 379.5 -> 372.1 mm, vias 7 -> 10
- net Net-(c5_6-Pad15): track 45.8 -> 50.2 mm
- net Net-(c1_2-Pad15): track 92.7 -> 97.1 mm
- net +3V3: track 229.6 -> 234.0 mm, vias 0 -> 9
- net Net-(c5_6-Pad16): track 33.0 -> 36.5 mm
- net Net-(c7_8-Pad13): track 124.7 -> 127.9 mm
- net Net-(c5_6-Pad4): track 87.9 -> 90.4 mm
- net Net-(c3_4-Pad13): track 103.1 -> 105.6 mm
- net Net-(c5_6-Pad14): track 39.9 -> 42.1 mm
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- added copper zone on F.Cu, net GND
Other:
- board outline added: 142.2 x 64.8 mm
- net class Default: trace_width 0.25 -> 0.5; via_dia 0.8 -> 1.1; via_drill 0.4 -> 0.6
- net class thick added: clearance 0.5, trace_width 1.25, via_dia 1.25, via_drill 0.6
- board text added: "3.3V"
- board text added: "5V"
- board text added: "P1"
- board text added: "P2"
- board text added: "P4"
- board text added: "P5"
- board text added: "P6"
- board text added: "P7"
- board text added: "P8"
- board text added: "p3"
