File: 8xrj45.sch (KiCad schematic (older format))
At the start: 5 parts, among them j1 Conn_01x40

Commit message: v2 design
Changed lines of the file:
@@
-$EndComp
-$Comp
-L power:GND #PWR0126
-U 1 1 5E55E241
-P 4750 1750
-F 0 "#PWR0126" H 4750 1500 50  0001 C CNN
-F 1 "GND" H 4755 1577 50  0000 C CNN
-F 2 "" H 4750 1750 50  0001 C CNN
-F 3 "" H 4750 1750 50  0001 C CNN
-	1    4750 1750
-	1    0    0    -1
 $EndComp
 $Comp
@@
 	4450 1750 4450 1600
 Wire Wire Line
-	4750 1750 4750 1600
-Wire Wire Line
 	5250 1750 5250 1600
 Wire Wire Line
@@
 Wire Wire Line
 	10100 3000 10100 5200
+Wire Wire Line
+	4750 1600 4750 1750
+$Comp
+L power:GND #PWR?
+U 1 1 5F61E395
+P 4750 1750
+F 0 "#PWR?" H 4750 1500 50  0001 C CNN
+F 1 "GND" H 4755 1577 50  0000 C CNN
+F 2 "" H 4750 1750 50  0001 C CNN
+F 3 "" H 4750 1750 50  0001 C CNN
+	1    4750 1750
+	1    0    0    -1
+$EndComp
 $EndSCHEMATC
